File: v2.0/Top/OtterIron_PRO_Top.sch (KiCad schematic (older format))
At the start: 33 parts, among them J1 USB_C_Receptacle_USB2.0, J10 Conn_01x01, J11 Conn_01x01, J12 Conn_01x01, J13 Conn_01x01, J14 Conn_01x01, J15 Conn_01x01, J16 Conn_01x01, J2 OLED_64x32, J3 Conn_01x01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

Commit message: add reset
Parts:
- U1: symbol Power_Protection:USBLC6-2SC6 -> OtterIron_PRO_Top-rescue:USBLC6-2SC6-Power_Protection
- U3: symbol otter:STUSB4500 -> OtterIron_PRO_Top-rescue:STUSB4500-otter
Changed lines of the file:
@@
 EESchema Schematic File Version 4
-LIBS:OtterIron_PRO_Top-cache
 EELAYER 30 0
 EELAYER END
@@
 	8050 2800 9150 2800
 $Comp
-L Power_Protection:USBLC6-2SC6 U1
+L OtterIron_PRO_Top-rescue:USBLC6-2SC6-Power_Protection U1
 U 1 1 5BF3991B
 P 3450 3350
@@
 Connection ~ 3500 7850
 $Comp
-L otter:STUSB4500 U3
+L OtterIron_PRO_Top-rescue:STUSB4500-otter U3
 U 1 1 5CE79B83
 P 4300 7900
